File: pcb/arch_40.kicad_pcb (KiCad board)
At the start: 2 copper layers, 275.5 x 130.3 mm, 104 parts, among them SW0-1 SWITCH_PUSH, SW0-2 SWITCH_PUSH, SW0-3 SWITCH_PUSH, SW0-4 SWITCH_PUSH, SW1-1 SWITCH_PUSH, SW1-2 SWITCH_PUSH, SW1-3 SWITCH_PUSH, SW10-1 SWITCH_PUSH, SW10-2 SWITCH_PUSH, SW10-3 SWITCH_PUSH, SW10-4 SWITCH_PUSH, SW11-1 SWITCH_PUSH, SW11-2 SWITCH_PUSH, SW11-3 SWITCH_PUSH, SW12-1 SWITCH_PUSH, SW12-2 SWITCH_PUSH, SW12-3 SWITCH_PUSH, SW12-4 SWITCH_PUSH, SW2-1 SWITCH_PUSH, SW2-2 SWITCH_PUSH, SW2-3 SWITCH_PUSH, SW2-4 SWITCH_PUSH, SW3-1 SWITCH_PUSH, SW3-2 SWITCH_PUSH, SW3-3 SWITCH_PUSH, SW3-4 SWITCH_PUSH, SW4-1 SWITCH_PUSH, SW4-2 SWITCH_PUSH, SW4-3 SWITCH_PUSH, SW4-4 SWITCH_PUSH, SW5-1 SWITCH_PUSH, SW5-2 SWITCH_PUSH, SW5-3 SWITCH_PUSH, SW5-4 SWITCH_PUSH, SW6-1 SWITCH_PUSH, SW6-2 SWITCH_PUSH, SW6-3 SWITCH_PUSH, SW7-1 SWITCH_PUSH, SW7-2 SWITCH_PUSH, SW7-3 SWITCH_PUSH, SW7-4 SWITCH_PUSH, SW8-1 SWITCH_PUSH, SW8-2 SWITCH_PUSH, SW8-3 SWITCH_PUSH, SW8-4 SWITCH_PUSH, SW9-1 SWITCH_PUSH, SW9-2 SWITCH_PUSH, SW9-3 SWITCH_PUSH, SW9-4 SWITCH_PUSH, U1 ARDUINO_PRO_MICRO

Commit message: fixed cutout.
Parts:
- moved D11-3 9.19 mm to (256.1, 84.9), turned to 105 degrees
Routing:
- net /COL11: track 172.8 -> 152.8 mm
- net /ROW-4: track 340.7 -> 353.5 mm
- net Net-(D11-3-Pad1): track 3.32 -> 11.6 mm
- net /ROW-3: track 407.7 -> 404.2 mm
Other:
- outline, holes or cut-outs redrawn

Commit message: updated pcb rev1
Parts:
- moved D1-3 0.69 mm to (45.1, 92.8)
- moved D0-4 0.61 mm to (16.8, 104.9)
- moved D6-3 0.60 mm to (129.1, 152.2)
- moved D2-4 0.55 mm to (62.4, 107.2)
- moved D10-4 0.53 mm to (234.6, 106.4)
- moved D9-4 0.40 mm to (213.7, 107.2)
- moved D12-4 0.39 mm to (277.1, 104.9)
- moved D6-1 0.39 mm to (173.0, 155.7)
Other:
- board size 275.5 x 130.3 mm -> 284.2 x 131 mm

Commit message: updated pcb rev1.1
Parts:
- SW0-1, SW0-2, SW0-3, SW0-4, SW12-1, SW12-2, SW12-3, SW12-4: footprint mxalpshybrid:MXOnly-1.5U-NoLED -> keebio_footprints:MX-Alps-Choc-1U-NoLED
- SW1-1, SW1-2, SW1-3, SW10-1, SW10-2, SW10-3, SW10-4, SW11-1, SW11-2, SW11-3, SW2-1, SW2-2, SW2-3, SW2-4, SW3-1, SW3-2, SW3-3, SW3-4, SW4-1, SW4-2, SW4-3, SW4-4, SW5-1, SW5-2, SW5-3, SW5-4, SW6-1, SW6-2, SW7-1, SW7-2, SW7-3, SW7-4, SW8-1, SW8-2, SW8-3, SW8-4, SW9-1, SW9-2, SW9-3, SW9-4: footprint mxalpshybrid:MXOnly-1U-NoLED -> keebio_footprints:MX-Alps-Choc-1U-NoLED
- SW6-3: footprint mxalpshybrid:MXOnly-2U-NoLED -> keebio_footprints:MX-Alps-Choc-2U-StabNormal-noled-alt
- moved D11-3 10.1 mm to (249.5, 92.6), turned to 15 degrees
Connections:
- U1 pad 2: (no net) -> Net-(U1-Pad2)
- U1 pad 21: (no net) -> VCC
- U1 pad 24: (no net) -> Net-(U1-Pad24)
Routing:
- net /ROW-4: track 353.5 -> 559.4 mm, vias 0 -> 4
- net /ROW-2: track 361.7 -> 533.1 mm, vias 0 -> 1
- net /ROW-1: track 288.9 -> 422.6 mm, vias 0 -> 1
- net /ROW-3: track 404.2 -> 499.1 mm, vias 1 -> 3
- net /COL11: track 152.8 -> 175.7 mm, vias 0 -> 1
- net /COL12: track 213.9 -> 226.1 mm, vias 0 -> 1
- net /COL4: track 105.3 -> 117.1 mm, vias 0 -> 1
- net Net-(D7-2-Pad1): track 3.29 -> 14.0 mm
- net Net-(D2-2-Pad1): track 3.98 -> 12.4 mm
- net Net-(D5-3-Pad1): track 3.56 -> 11.8 mm
- net Net-(D7-1-Pad1): track 3.24 -> 11.4 mm
- net Net-(D5-2-Pad1): track 3.45 -> 11.5 mm
- net Net-(D12-3-Pad1): track 3.48 -> 11.5 mm
- net Net-(D0-4-Pad1): track 3.95 -> 11.4 mm
- net Net-(D1-1-Pad1): track 3.83 -> 11.3 mm
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Other:
- outline, holes or cut-outs redrawn
- board text added: "Arch40 rev 1.1"
